File: pcb/weather.kicad_sch (KiCad schematic)
At the start: 7 parts, among them J1 dht11, J2 EXTRA PINS, J3 Conn_01x02_Pin, U2 TFT_ST7735_SD, U3 WEMOS_C3_Mini

Commit message: Add files via upload
Connections:
- net +3.3V: now also U2.1 (3V3)
- net GND: now also U2.2 (GND)
Other:
- moved on the sheet: J1, J2, J3, R1, U1, U2, U3
