File: pcb/weather.kicad_pcb (KiCad board)
At the start: 2 copper layers, 50 x 75 mm, 27 parts, among them J1 dht11, J2 EXTRA PINS, J3 Conn_01x02_Pin, U2 TFT_ST7735_SD, U3 WEMOS_C3_Mini

Commit message: Add files via upload
Parts:
- moved REF** 23.1 mm to (152.5, 87.5)
- moved G*** 22.1 mm to (152.5, 60.8) (x2)
- moved G*** 22.1 mm to (172.7, 34.4) (x2)
- moved G*** 22.1 mm to (194.1, 43.8)
- moved G*** 22.1 mm to (192.5, 35.4) (x2)
- moved G*** 22.1 mm to (159.7, 68.4)
- moved G*** 22.1 mm to (177.1, 68.2)
- moved G*** 22.1 mm to (194.1, 60.6)
- moved G*** 22.1 mm to (152.8, 37.0)
- moved J2 22.1 mm to (152.2, 49.0)
- moved J3 22.1 mm to (173.5, 86.2)
- moved REF** 22.1 mm to (151.8, 94.0)
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Connections:
- U2 pad 1: unconnected-(U2-3V3-Pad1) -> VCC
- U2 pad 2: unconnected-(U2-GND-Pad2) -> GND
Routing:
- net MISO: track 96.9 -> 84.3 mm
- net IO4: track 27.6 -> 25.9 mm, vias 1 -> 3

Commit message: pcb did
Parts:
- removed the G*** at (194.1, 43.8)
- removed the G*** at (159.7, 68.4)
- removed the G*** at (177.1, 68.2)
- removed the G*** at (194.1, 60.6)
- removed the G*** at (152.8, 37.0)
- removed the REF** at (159.9, 94.0)
- removed the REF** at (156.0, 100.2) (x2)
- removed the REF** at (174.5, 73.4)
- removed the REF** at (151.8, 94.0)
- G*** (x2): moved to B.Cu
- moved G*** 86.5 mm to (209.1, -4.67), turned to 180 degrees (x2)
- moved J2 16.8 mm to (151.8, 32.2), turned to 90 degrees
- moved REF** 7.04 mm to (152.5, 101.0)
Routing:
- net MISO: track 84.3 -> 63.7 mm
- net IO5: track 10.9 -> 28.9 mm, vias 0 -> 1
- net IO4: track 25.9 -> 43.6 mm, vias 3 -> 4
- net IO1: track 10.7 -> 20.2 mm
Other:
- board text added: "Souptik Samanta Souptik.me"
- board text removed: "Methamphetamine"
- board text removed: "Souptik Samanta @04-09-2009"
- board text removed: "Souptik Samanta Souptik@souptik.me"
